File: Plate Right/ergocape.sch (KiCad schematic (older format))
At the start: 43 parts

Commit message: cleanup and finish the case files
Parts:
- removed K_ESC1: KEYSW, acheron_SwitchSlots:slotMX100, symbol keyboard_parts:KEYSW
- added K_BKSP_1: KEYSW, usbc_footprint:slotMX200, symbol keyboard_parts:KEYSW
- H1, H10, H11, H12, H2, H3, H5, H6, H8, H9: footprint usbc_footprint:mount_hole_2.4x4 -> acheron_MountingHoles:MountingHole_2.5x4.0mm
- K_1, K_2, K_3, K_4, K_5, K_A1, K_ALT1, K_B1, K_BOT_1U_1, K_BOT_1U_2, K_C1, K_CTRL1, K_D1, K_E1, K_F1, K_G1, K_Q1, K_R1, K_S1, K_T1, K_TAB1, K_THUMB_1U_3, K_THUMB_1U_4, K_TH_1U_1, K_TH_1U_2, K_V1, K_W1, K_WIN1, K_X1, K_Z1: footprint acheron_SwitchSlots:slotMX100 -> usbc_footprint:slotMX100
- K_ENTER_rev_2.25u_1, K_SHIFT_REV_2.75_1: footprint acheron_SwitchSlots:slotMX200 -> usbc_footprint:slotMX200
Connections:
- wire segments 3 -> 1
