File: Plate Left_2u/ergocape.kicad_pcb (KiCad board)
At the start: 2 copper layers, 183.2 x 140.8 mm, 43 parts

Commit message: fix pro micro footprint
Parts:
- removed the REF** at (52.6, 21.8) (x2)
- added K_XTRA1: KEYSW, usbc_footprint:1u_uni, F.Cu at (46.1, 39.7)
- added REF**: OSHW-Logo2_9.8x8mm_SilkScreen, logo_lib:OSHW-Logo2_9.8x8mm_SilkScreen, B.Cu at (56.1, 21.6)
- added REF**: OSHW-Logo2_9.8x8mm_SilkScreen, logo_lib:OSHW-Logo2_9.8x8mm_SilkScreen, F.Cu at (56.1, 21.6)
- K_ESC1: footprint usbc_footprint:mixed_2u_uni_centered -> usbc_footprint:1u_uni
- moved K_ESC1 9.46 mm to (65.1, 39.7)
- moved K_TH_1U_1 0.22 mm to (191.9, 127.9)
- moved H8 0.22 mm to (179.6, 132.9)
- moved K_THUMB_2U1 0.22 mm to (170.6, 128.5)
- moved K_TH_1U_2 0.22 mm to (183.9, 145.2)
Other:
- board size 183.2 x 140.8 mm -> 186.4 x 145 mm
- board text added: ""Tazz""
- board text added: "captn3m0"
- board text added: "created by u/Harshitgoel96"
- board text added: "u/Delta_Two"
- board text added: "u/Senor_Goobe"
- board text removed: "For the love of Keycaps"
